File: 65_keyboard/65_keyboard.kicad_sch (KiCad schematic)
At the start: 141 parts, among them SW1 MX_SW_solder, SW10 MX_SW_solder, SW11 MX_SW_solder, SW12 MX_SW_solder, SW13 MX_SW_solder, SW14 MX_SW_solder, SW15 MX_SW_solder, SW16 MX_SW_solder, SW17 MX_SW_solder, SW18 MX_SW_solder, SW19 MX_SW_solder, SW2 MX_SW_solder, SW20 MX_SW_solder, SW21 MX_SW_solder, SW22 MX_SW_solder, SW23 MX_SW_solder, SW24 MX_SW_solder, SW25 MX_SW_solder, SW26 MX_SW_solder, SW27 MX_SW_solder, SW28 MX_SW_solder, SW29 MX_SW_solder, SW3 MX_SW_solder, SW30 MX_SW_solder, SW31 MX_SW_solder, SW32 MX_SW_solder, SW33 MX_SW_solder, SW34 MX_SW_solder, SW35 MX_SW_solder, SW36 MX_SW_solder, SW37 MX_SW_solder, SW38 MX_SW_solder, SW39 MX_SW_solder, SW4 MX_SW_solder, SW40 MX_SW_solder, SW41 MX_SW_solder, SW42 MX_SW_solder, SW43 MX_SW_solder, SW44 MX_SW_solder, SW45 MX_SW_solder, SW46 MX_SW_solder, SW47 MX_SW_solder, SW48 MX_SW_solder, SW49 MX_SW_solder, SW5 MX_SW_solder, SW50 MX_SW_solder, SW51 MX_SW_solder, SW52 MX_SW_solder, SW53 MX_SW_solder, SW54 MX_SW_solder, SW55 MX_SW_solder, SW56 MX_SW_solder, SW57 MX_SW_solder, SW58 MX_SW_solder, SW59 MX_SW_solder, SW6 MX_SW_solder, SW60 MX_SW_solder, SW61 MX_SW_solder, SW62 MX_SW_solder, SW63 MX_SW_solder, SW64 MX_SW_solder, SW65 MX_SW_solder, SW66 MX_SW_solder, SW67 MX_SW_solder, SW68 MX_SW_solder, SW7 MX_SW_solder, SW8 MX_SW_solder, SW9 MX_SW_solder, U1 Seeeduino Xiao nRF52840

Commit message: Done with schematics
Parts:
- added BT2: BK-18650-PC2, BK-18650-PC2:BAT_BK-18650-PC2, symbol BK-18650-PC2:BK-18650-PC2
- added J1, J2: Conn_01x06_Pin, Connector_PinHeader_2.54mm:PinHeader_1x06_P2.54mm_Vertical, symbol Connector:Conn_01x06_Pin
- added U2, U3: 74HC595, Package_DIP:DIP-16_W7.62mm, symbol 74xx:74HC595
- U1: value Seeeduino Xiao nRF52840 -> Xiao nRF52840
Connections:
- net Col9: now reaches SW63.1
- net Col9: now also SW10.1, SW25.1, SW40.1, SW54.1, U3.1 (QB)
- net at SW2.2: now also D2.2 (A); no longer D2.1 (K)
- net at SW26.1: now also SW11.1, SW41.1, SW55.1, SW64.1
- net row4: now reaches D60.1 (K)
- net row4: now also D59.1 (K), D61.1 (K), D62.1 (K), D63.1 (K), D64.1 (K), D65.1 (K), D66.1 (K), D67.1 (K), D68.1 (K), U1.14 (P1.12)
- net Col6: now reaches SW22.1
- net Col6: now also SW37.1, SW51.1, SW7.1, U2.6 (QG)
- net row2: now reaches D40.1 (K)
- net row2: now also D31.1 (K), D32.1 (K), D33.1 (K), D34.1 (K), D35.1 (K), D36.1 (K), D37.1 (K), D38.1 (K), D39.1 (K), D41.1 (K), D42.1 (K), D43.1 (K), D44.1 (K), U1.4 (P0.29)
- net Col1: now reaches SW17.1
- net Col1: now also SW2.1, SW32.1, SW46.1, SW60.1, U2.1 (QB)
- net Col8: now reaches SW24.1
- net Col8: now also SW39.1, SW53.1, SW9.1, U3.15 (QA)
- net Col2: now reaches SW18.1
- net Col2: now also SW3.1, SW33.1, SW47.1, SW61.1, U2.2 (QC)
- net row0: now reaches D11.1 (K)
- net row0: now also D1.1 (K), D10.1 (K), D12.1 (K), D13.1 (K), D14.1 (K), D15.1 (K), D2.1 (K), D3.1 (K), D4.1 (K), D5.1 (K), D6.1 (K), D7.1 (K), D8.1 (K), D9.1 (K), U1.2 (P0.03)
- net row3: now reaches D51.1 (K)
- net row3: now also D45.1 (K), D46.1 (K), D47.1 (K), D48.1 (K), D49.1 (K), D50.1 (K), D52.1 (K), D53.1 (K), D54.1 (K), D55.1 (K), D56.1 (K), D57.1 (K), D58.1 (K), U1.7 (P1.11)
- net row1: now reaches D21.1 (K)
- net row1: now also D16.1 (K), D17.1 (K), D18.1 (K), D19.1 (K), D20.1 (K), D22.1 (K), D23.1 (K), D24.1 (K), D25.1 (K), D26.1 (K), D27.1 (K), D28.1 (K), D29.1 (K), D30.1 (K), U1.3 (P0.28)
- net Col0: now reaches SW31.1
- net Col0: now also SW1.1, SW16.1, SW45.1, SW59.1, U2.15 (QA)
- net Col3: now reaches SW48.1
- net Col3: now also SW19.1, SW34.1, SW4.1, U2.3 (QD)
- net Col14: now reaches SW44.1
- net Col14: now also SW15.1, SW30.1, SW58.1, SW68.1, U3.6 (QG)
- net Col12: now reaches SW13.1
- net Col12: now also SW28.1, SW43.1, SW56.1, SW66.1, U3.4 (QE)
- net Col4: now reaches SW5.1
- net Col4: now also SW20.1, SW35.1, SW49.1, U2.4 (QE)
- net Col13: now reaches SW67.1
- net Col13: now also SW14.1, SW29.1, SW57.1, U3.5 (QF)
- net Col5: now reaches SW50.1
- net Col5: now also SW21.1, SW36.1, SW6.1, SW62.1, U2.5 (QF)
- net Col11: now reaches SW27.1
- net Col11: now also SW12.1, SW42.1, SW65.1, U3.3 (QD)
- net Col7: now reaches SW52.1
- net Col7: now also SW23.1, SW38.1, SW8.1, U2.7 (QH)
- net D1: now reaches U1.1 (P0.02)
- net D1: now also U2.12 (RCLK), U3.12 (RCLK)
- net +3.3V: now reaches U1.10 (3V3)
- net +3.3V: now also J1.1 (Pin_1), U2.10 (~{SRCLR}), U2.16 (VCC), U3.10 (~{SRCLR}), U3.16 (VCC)
- net SER: now reaches U1.11 (P1.15)
- net SER: now also U2.14 (SER)
- net RST: now reaches U1.12 (P1.14)
- net RST: now also J1.5 (Pin_5)
- net SCK: now reaches U1.13 (P1.13)
- net SCK: now also U2.11 (SRCLK), U3.11 (SRCLK)
- net BAT-: now reaches U1.15 (BAT-)
- net BAT-: now also BT2.-
- net BAT+: now reaches U1.16 (BAT+)
- net BAT+: now also BT2.+
- net BUSY: now reaches U1.17 (P0.09)
- net BUSY: now also J1.6 (Pin_6)
- net SDA: now reaches U1.5 (P0.04)
- net SDA: now also J1.3 (Pin_3)
- net SCL: now reaches U1.6 (P0.05)
- net SCL: now also J1.4 (Pin_4)
- net GND: now reaches U1.9 (GND)
- net GND: now also J1.2 (Pin_2), U2.13 (~{OE}), U2.8 (GND), U3.13 (~{OE}), U3.8 (GND)
- new net: U2.9 (QH'), U3.14 (SER)
- new net Col10: U3.2 (QC)
- no-connect marks 0 -> 1
Other:
- note added: "1.9" E-Paper Display(for vibes)"
- note added: "18650 Cell"
- note added: "Shift Registers"
- note added: "Switches w/Diodes"
- moved on the sheet: D2, D31, D32, D33, D34, D35, D36, D37, D38, D39, D40, D41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
